Commit message: updated laser_joint origin

File: description/lidar.xacro (robot description, xacro)
@@ -4,5 +4,5 @@
         <parent link="chassis"/>
         <child link="laser_frame"/>
-        <origin xyz="0.1 0 0.175" rpy="0 0 0"/>
+        <origin xyz="0.115 0 0.075" rpy="0 0 0"/>
         <!--         CHANGE THIS           -->
     </joint>
