Commit message: Modifed robot_core_xacro to be Roberto's bot UDRF

File: description/robot_core.xacro (robot description, xacro)
@@ -9,6 +9,9 @@
         <color rgba="0 0 0 1"/>
     </material>
-    <material name="blue">
-        <color rgba="0.5 0.5 1 1"/>
+    <material name="white">
+        <color rgba="1 1 1 1"/>
+    </material>
+    <material name="transparent_yellow">
+        <color rgba="1 1 0 0.6"/>
     </material>
     <!-- BASE LINK -->
@@ -19,23 +22,37 @@
         <parent link="base_link"/>
         <child link="chassis"/>
-        <origin xyz="-0.1 0 0"/>
+        <origin xyz="-0.022 0 0"/>
     </joint>
     <link name="chassis">
         <visual>
-            <origin xyz="0.15 0 0.075"/>
+            <origin xyz="0.115 0 0"/>
             <geometry>
-                <box size="0.3 0.3 0.15"/>
+                <box size="0.23 0.14 0.04"/>
             </geometry>
             <material name="red"/>
         </visual>
         <collision>
-            <origin xyz="0.15 0 0.075"/>
+            <origin xyz="0.115 0 0"/>
             <geometry>
-                <box size="0.3 0.3 0.15"/>
+                <box size="0.23 0.14 0.04"/>
             </geometry>
         </collision>
-        <xacro:inertial_box mass="0.5" x="0.3" y="0.3" z="0.15">
-            <origin xyz="0.15 0 0.075" rpy="0 0 0"/>
+        <xacro:inertial_box mass="0.5" x="0.23" y="0.14" z="0">
+            <origin xyz="0.115 0 0" rpy="0 0 0"/>
         </xacro:inertial_box>
+    </link>
+    <!-- YELLOW BOX ON TOP -->
+    <joint name="yellow_box_on_top_joint" type="fixed">
+        <parent link="chassis"/>
+        <child link="yellow_box_on_top"/>
+    </joint>
+    <link name="yellow_box_on_top">
+        <visual>
+            <origin xyz="0.11 0 0.06"/>
+            <geometry>
+                <box size="0.075 0.075 0.075"/>
+            </geometry>
+            <material name="transparent_yellow"/>
+        </visual>
     </link>
     <!-- LEFT WHEEL LINK -->
@@ -43,5 +60,5 @@
         <parent link="base_link"/>
         <child link="left_wheel"/>
-        <origin xyz="0 0.175 0" rpy="-${pi/2} 0 0"/>
+        <origin xyz="0 0.09 0" rpy="-${pi/2} 0 0"/>
         <axis xyz="0 0 1"/>
     </joint>
@@ -49,5 +66,5 @@
         <visual>
             <geometry>
-                <cylinder radius="0.05" length="0.04"/>
+                <cylinder radius="0.045" length="0.04"/>
             </geometry>
             <material name="black"/>
@@ -55,8 +72,8 @@
         <collision>
             <geometry>
-                <cylinder radius="0.05" length="0.04"/>
+                <cylinder radius="0.045" length="0.04"/>
             </geometry>
         </collision>
-        <xacro:inertial_cylinder mass="0.1" length="0.84" radius="0.05">
+        <xacro:inertial_cylinder mass="0.1" length="0.04" radius="0.045">
             <origin xyz="0 0 0" rpy="0 0 0"/>
         </xacro:inertial_cylinder>
@@ -66,5 +83,5 @@
         <parent link="base_link"/>
         <child link="right_wheel"/>
-        <origin xyz="0 -0.175 0" rpy="${pi/2} 0 0"/>
+        <origin xyz="0 -0.09 0" rpy="${pi/2} 0 0"/>
         <axis xyz="0 0 -1"/>
     </joint>
@@ -72,5 +89,5 @@
         <visual>
             <geometry>
-                <cylinder radius="0.05" length="0.04"/>
+                <cylinder radius="0.045" length="0.04"/>
             </geometry>
             <material name="black"/>
@@ -78,8 +95,8 @@
         <collision>
             <geometry>
-                <cylinder radius="0.05" length="0.04"/>
+                <cylinder radius="0.045" length="0.04"/>
             </geometry>
         </collision>
-        <xacro:inertial_cylinder mass="0.1" length="0.84" radius="0.05">
+        <xacro:inertial_cylinder mass="0.1" length="0.04" radius="0.045">
             <origin xyz="0 0 0" rpy="0 0 0"/>
         </xacro:inertial_cylinder>
@@ -89,19 +106,19 @@
         <parent link="chassis"/>
         <child link="caster_wheel"/>
-        <origin xyz="0.24 0 0"/>
+        <origin xyz="0.2 0 -0.0225"/>
     </joint>
     <link name="caster_wheel">
         <visual>
             <geometry>
-                <sphere radius="0.05"/>
+           <sphere radius="0.025"/>
             </geometry>
-            <material name="blue"/>
+            <material name="white"/>
         </visual>
         <collision>
             <geometry>
-                <sphere radius="0.05"/>
+                <sphere radius="0.025"/>
             </geometry>
         </collision>
-        <xacro:inertial_sphere mass="0.1" radius="0.05">
+        <xacro:inertial_sphere mass="0.1" radius="0.025">
             <origin xyz="0 0 0" rpy="0 0 0"/>
         </xacro:inertial_sphere>

Commit message: Created core URDF

File: description/robot_core.xacro (robot description, xacro)
@@ -12,6 +12,6 @@
         <color rgba="1 1 1 1"/>
     </material>
-    <material name="transparent_yellow">
-        <color rgba="1 1 0 0.6"/>
+    <material name="transparent_white">
+        <color rgba="1 1 1 0.5"/>
     </material>
     <!-- BASE LINK -->
@@ -42,16 +42,16 @@
         </xacro:inertial_box>
     </link>
-    <!-- YELLOW BOX ON TOP -->
-    <joint name="yellow_box_on_top_joint" type="fixed">
+    <!-- WHITE BOX ON TOP -->
+    <joint name="white_box_on_top_joint" type="fixed">
         <parent link="chassis"/>
-        <child link="yellow_box_on_top"/>
+        <child link="white_box_on_top"/>
     </joint>
-    <link name="yellow_box_on_top">
+    <link name="white_box_on_top">
         <visual>
-            <origin xyz="0.11 0 0.06"/>
+            <origin xyz="0.11 0 0.0575"/>
             <geometry>
-                <box size="0.075 0.075 0.075"/>
+                <box size="0.1 0.075 0.075"/>
             </geometry>
-            <material name="transparent_yellow"/>
+            <material name="transparent_white"/>
         </visual>
     </link>

Commit message: added BASE footprint joint and link

File: description/robot_core.xacro (robot description, xacro)
@@ -17,4 +17,12 @@
     <!-- BASE LINK -->
     <link name="base_link">
+    </link>
+    <!-- BASE FOOTPRINT LINK -->
+    <joint name="base_footprint_joint" type="fixed">
+        <parent link="base_link"/>
+        <child link="base_footprint"/>
+        <origin xyz="0 0 0" rpy="0 0 0"/>
+    </joint>
+    <link name="base_footprint">
     </link>
     <!-- CHASSIS LINK -->

Commit message: added gz tag for friction

File: description/robot_core.xacro (robot description, xacro)
@@ -114,5 +114,5 @@
         <parent link="chassis"/>
         <child link="caster_wheel"/>
-        <origin xyz="0.2 0 -0.0225"/>
+        <origin xyz="0.2 0 -0.0165"/>
     </joint>
     <link name="caster_wheel">
@@ -132,3 +132,7 @@
         </xacro:inertial_sphere>
     </link>
+    <gazebo reference="caster_wheel">
+        <mu1 value="0.001"/>
+        <mu2 value="0.001"/>
+    </gazebo>
 </robot>
